File: KiCad_PCB_Ornament/Ornament.kicad_pcb (KiCad board)
At the start: 2 copper layers, 99 x 117.7 mm, 55 parts, among them J1 Conn_01x04_Pin, J2 Conn_01x04_Pin, Q1 TEMT6200FX01, SW1 SW_Push, SW2 SW_SPDT, U1 ATtiny414-SS, U2 INA190A3IDDFR

Commit message: PCB updates to fix current sense amplifier layout and complete BOM
Connections:
- U2 pad 1: PB1 -> VCC
- U2 pad 2: (no net) -> VCC
- U2 pad 3: (no net) -> GND
- U2 pad 5: VCC -> PB1
- U2 pad 6: GND -> unconnected-(U2-NC-Pad6)
- U2 pad 7: Net-(U2--) -> Net-(U2-+)
- U2 pad 8: Net-(U2-+) -> Net-(U2--)
Routing:
- net Net-(U2-+): track 3.84 -> 8.25 mm, vias 0 -> 2
- net GND: track 12.4 -> 8.15 mm, vias 74 -> 73
- net VCC: track 26.4 -> 29.6 mm
- net PB1: track 4.72 -> 7.66 mm, vias 0 -> 2
- net Net-(U2--): track 3.96 -> 4.57 mm
Changed lines of the file:
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@@
 	(net 26 "Net-(U2-+)")
 	(net 27 "Net-(U2--)")
+	(net 28 "unconnected-(U2-NC-Pad6)")
 	(footprint "LED_SMD:LED_0603_1608Metric_Pad1.05x0.95mm_HandSolder"
 		(layer "F.Cu")
@@
 			(layers "F.Cu" "F.Mask" "F.Paste")
 			(roundrect_rratio 0.25)
-			(net 22 "PB1")
-			(pintype "output")
+			(net 4 "VCC")
+			(pinfunction "VS")
+			(pintype "power_in")
 		)
 		(pad "2" smd roundrect
@@
 			(layers "F.Cu" "F.Mask" "F.Paste")
 			(roundrect_rratio 0.25)
+			(net 4 "VCC")
+			(pinfunction "Enable")
+			(pintype "input")
 		)
 		(pad "3" smd roundrect
@@
 			(layers "F.Cu" "F.Mask" "F.Paste")
 			(roundrect_rratio 0.25)
+			(net 1 "GND")
+			(pinfunction "REF")
+			(pintype "input")
 		)
 		(pad "4" smd roundrect
@@
 			(roundrect_rratio 0.25)
 			(net 1 "GND")
-			(pinfunction "REF")
-			(pintype "input")
+			(pinfunction "GND")
+			(pintype "power_in")
 		)
 		(pad "5" smd roundrect
@@
 			(layers "F.Cu" "F.Mask" "F.Paste")
 			(roundrect_rratio 0.25)
-			(net 4 "VCC")
-			(pinfunction "V+")
-			(pintype "power_in")
+			(net 22 "PB1")
+			(pintype "output")
 		)
 		(pad "6" smd roundrect
@@
 			(layers "F.Cu" "F.Mask" "F.Paste")
 			(roundrect_rratio 0.25)
-			(net 1 "GND")
-			(pinfunction "GND")
-			(pintype "power_in")
+			(net 28 "unconnected-(U2-NC-Pad6)")
+			(pinfunction "NC")
+			(pintype "no_connect")
 		)
 		(pad "7" smd roundrect
@@
 			(layers "F.Cu" "F.Mask" "F.Paste")
 			(roundrect_rratio 0.25)
-			(net 27 "Net-(U2--)")
-			(pinfunction "-")
+			(net 26 "Net-(U2-+)")
+			(pinfunction "+")
 			(pintype "input")
 		)
@@
 			(layers "F.Cu" "F.Mask" "F.Paste")
 			(roundrect_rratio 0.25)
-			(net 26 "Net-(U2-+)")
-			(pinfunction "+")
+			(net 27 "Net-(U2--)")
+			(pinfunction "-")
 			(pintype "input")
 		)
@@
 	)
 	(segment
-		(start 98.157 125.7055)
-		(end 99.1845 125.7055)
-		(width 0.2)
-		(layer "F.Cu")
-		(net 1)
-	)
-	(segment
-		(start 99.329 125.85)
-		(end 99.445 125.966)
-		(width 0.2)
-		(layer "F.Cu")
-		(net 1)
-	)
-	(segment
-		(start 99.445 125.966)
-		(end 99.445 126.558)
-		(width 0.2)
+		(start 89.29 129.902)
+		(end 91.829496 129.902)
+		(width 0.5)
 		(layer "F.Cu")
 		(net 1)
 	)
 	(segment
-		(start 99.445 126.558)
-		(end 99.626 126.739)
-		(width 0.2)
+		(start 95.457 126.274496)
+		(end 95.457 125.7965)
+		(width 0.5)
 		(layer "F.Cu")
 		(net 1)
 	)
 	(segment
-		(start 99.1845 125.7055)
-		(end 99.329 125.85)
-		(width 0.2)
+		(start 91.829496 129.902)
+		(end 95.457 126.274496)
+		(width 0.5)
 		(layer "F.Cu")
 		(net 1)
@@
 	)
 	(via
-		(at 99.626 126.739)
-		(size 0.6)
-		(drill 0.3)
-		(layers "F.Cu" "B.Cu")
-		(net 1)
-	)
-	(via
 		(at 90.253 118.799)
 		(size 0.6)
@@
 	)
 	(segment
-		(start 101.62742 132.967)
-		(end 102.927 132.967)
-		(width 0.2)
-		(layer "B.Cu")
-		(net 1)
-	)
-	(segment
-		(start 102.927 132.967)
-		(end 104.178 134.218)
-		(width 0.2)
-		(layer "B.Cu")
-		(net 1)
-	)
-	(segment
-		(start 99.626 130.96558)
-		(end 101.62742 132.967)
-		(width 0.2)
-		(layer "B.Cu")
-		(net 1)
-	)
-	(segment
-		(start 99.626 126.739)
-		(end 99.626 130.96558)
-		(width 0.2)
-		(layer "B.Cu")
-		(net 1)
-	)
-	(segment
 		(start 93.539 123.107)
 		(end 95.903 120.743)
@@
 	)
 	(segment
-		(start 98.2485 126.8095)
-		(end 99.056 127.617)
+		(start 95.457 124.3955)
+		(end 96.236999 124.3955)
 		(width 0.5)
 		(layer "F.Cu")
@@
 	)
 	(segment
-		(start 98.157 126.7004)
-		(end 98.157 126.3555)
-		(width 0.4006)
-		(layer "F.Cu")
-		(net 4)
-	)
-	(segment
-		(start 101.686 127.617)
-		(end 103.6435 125.6595)
+		(start 96.807 125.6339)
+		(end 96.807 126.708924)
 		(width 0.5)
 		(layer "F.Cu")
@@
 	)
 	(segment
-		(start 98.1564 126.3561)
-		(end 98.157 126.3555)
-		(width 0.4006)
-		(layer "F.Cu")
-		(net 4)
-	)
-	(segment
-		(start 98.2485 126.7919)
-		(end 98.2485 126.8095)
+		(start 105.398 125.6595)
+		(end 103.6435 125.6595)
 		(width 0.5)
 		(layer "F.Cu")
@@
 	)
 	(segment
-		(start 105.398 125.6595)
+		(start 101.686 127.617)
 		(end 103.6435 125.6595)
 		(width 0.5)
@@
 	)
 	(segment
-		(start 98.157 126.7004)
-		(end 98.2485 126.7919)
+		(start 95.457 124.9545)
+		(end 95.457 124.3955)
 		(width 0.5)
 		(layer "F.Cu")
@@
 	)
 	(segment
-		(start 99.056 127.617)
-		(end 101.686 127.617)
+		(start 96.788 125.6339)
+		(end 96.788 125.333076)
 		(width 0.5)
 		(layer "F.Cu")
@@
 	)
 	(segment
-		(start 96.807 125.6339)
-		(end 96.807 126.3183)
+		(start 96.409424 124.9545)
+		(end 95.457 124.9545)
 		(width 0.5)
 		(layer "F.Cu")
@@
 	)
 	(segment
-		(start 96.807 126.3183)
-		(end 96.8448 126.3561)
+		(start 96.807 126.708924)
+		(end 97.715076 127.617)
+		(width 0.5)
+		(layer "F.Cu")
+		(net 4)
+	)
+	(segment
+		(start 97.715076 127.617)
+		(end 101.686 127.617)
+		(width 0.5)
+		(layer "F.Cu")
+		(net 4)
+	)
+	(segment
+		(start 96.807 125.6339)
+		(end 96.788 125.6339)
 		(width 0.5)
 		(layer "F.Cu")
@@
 	)
 	(segment
-		(start 87.4048 118.8032)
-		(end 88.4715 118.8032)
+		(start 96.788 125.333076)
+		(end 96.409424 124.9545)
 		(width 0.5)
 		(layer "F.Cu")
@@
 	)
 	(segment
-		(start 96.8448 126.3561)
-		(end 98.1564 126.3561)
-		(width 0.4006)
+		(start 87.4048 118.8032)
+		(end 88.4715 118.8032)
+		(width 0.5)
 		(layer "F.Cu")
 		(net 4)
@@
 	)
 	(segment
-		(start 94.6237 124.3955)
-		(end 95.457 124.3955)
-		(width 0.2)
+		(start 98.157 126.427)
+		(end 98.497 126.767)
+		(width 0.4006)
 		(layer "F.Cu")
 		(net 22)
 	)
 	(segment
-		(start 94.064 124.9552)
-		(end 94.6237 124.3955)
-		(width 0.2)
+		(start 98.1564 126.3561)
+		(end 98.157 126.3555)
+		(width 0.4006)
 		(layer "F.Cu")
 		(net 22)
@@
 	)
 	(segment
-		(start 92.239 126.917)
-		(end 94.064 125.092)
-		(width 0.2)
+		(start 91.896 126.952)
+		(end 91.861 126.917)
+		(width 0.4006)
 		(layer "F.Cu")
 		(net 22)
 	)
 	(segment
-		(start 94.064 125.092)
-		(end 94.064 124.9552)
-		(width 0.2)
+		(start 98.157 126.3555)
+		(end 98.157 126.427)
+		(width 0.4006)
 		(layer "F.Cu")
 		(net 22)
 	)
 	(segment
+		(start 93.576 126.952)
+		(end 91.896 126.952)
+		(width 0.4006)
+		(layer "F.Cu")
+		(net 22)
+	)
+	(via
+		(at 98.497 126.767)
+		(size 0.6)
+		(drill 0.3)
+		(layers "F.Cu" "B.Cu")
+		(net 22)
+	)
+	(via
+		(at 93.576 126.952)
+		(size 0.6)
+		(drill 0.3)
+		(layers "F.Cu" "B.Cu")
+		(net 22)
+	)
+	(segment
+		(start 98.497 126.767)
+		(end 93.761 126.767)
+		(width 0.4006)
+		(layer "B.Cu")
+		(net 22)
+	)
+	(segment
+		(start 93.761 126.767)
+		(end 93.576 126.952)
+		(width 0.4006)
+		(layer "B.Cu")
+		(net 22)
+	)
+	(segment
 		(start 109.2907 122.6013)
 		(end 101.99 129.902)
@@
 	)
 	(segment
+		(start 99.458382 123.949642)
+		(end 100.264142 123.949642)
+		(width 0.3)
+		(layer "F.Cu")
+		(net 26)
+	)
+	(segment
+		(start 99.465 125.592918)
+		(end 99.465 126.767)
+		(width 0.3)
+		(layer "F.Cu")
+		(net 26)
+	)
+	(segment
+		(start 100.264142 123.949642)
+		(end 100.321 124.0065)
+		(width 0.3)
+		(layer "F.Cu")
+		(net 26)
+	)
+	(segment
 		(start 101.805 123.987)
 		(end 101.8185 123.9735)
@@
 	)
 	(segment
-		(start 98.5655 123.987)
-		(end 99.985 123.987)
-		(width 0.2)
+		(start 98.917582 125.0455)
+		(end 99.465 125.592918)
+		(width 0.3)
 		(layer "F.Cu")
 		(net 26)
 	)
 	(segment
-		(start 98.157 124.3955)
-		(end 98.5655 123.987)
-		(width 0.2)
+		(start 98.157 125.0455)
+		(end 98.917582 125.0455)
+		(width 0.3)
 		(layer "F.Cu")
 		(net 26)
 	)
+	(via
+		(at 99.458382 123.949642)
+		(size 0.6)
+		(drill 0.3)
+		(layers "F.Cu" "B.Cu")
+		(net 26)
+	)
+	(via
+		(at 99.465 126.767)
+		(size 0.6)
+		(drill 0.3)
+		(layers "F.Cu" "B.Cu")
+		(net 26)
+	)
 	(segment
-		(start 99.3185 125.0455)
-		(end 99.985 125.712)
-		(width 0.2)
+		(start 99.465 123.95626)
+		(end 99.458382 123.949642)
+		(width 0.3)
+		(layer "B.Cu")
+		(net 26)
+	)
+	(segment
+		(start 99.465 126.767)
+		(end 99.465 123.95626)
+		(width 0.3)
+		(layer "B.Cu")
+		(net 26)
+	)
+	(segment
+		(start 98.985 124.3955)
+		(end 98.157 124.3955)
+		(width 0.3)
 		(layer "F.Cu")
 		(net 27)
 	)
 	(segment
-		(start 98.157 125.0455)
-		(end 99.3185 125.0455)
-		(width 0.2)
+		(start 100.321 125.7315)
+		(end 98.985 124.3955)
+		(width 0.3)
 		(layer "F.Cu")
 		(net 27)
